File: Project/MicroMouse_2025_v2/MicroMouse_2025_v2.kicad_pcb (KiCad board)
At the start: 2 copper layers, 184.5 x 111.5 mm, 20 parts, among them J1 JST_HX-2, U1 RP2040-ZERO, U2 RP2040-Connect

Commit message: Added GY87 and DC DC Buck
Parts:
- added U10: ~, MicroMouse_2025_v2:GY-87, F.Cu at (176.8, 118.8)
- added U9: ~, MicroMouse_2025_v2:DC-DC 5V3A BEC, F.Cu at (203.1, 118.8)
Other:
- board size 184.5 x 111.5 mm -> 184.5 x 121.1 mm
