File: Project/MicroMouse_2025_v2/MicroMouse_2025_v2.kicad_sch (KiCad schematic)
At the start: 20 parts, among them J1 JST_HX-2, U1 RP2040-ZERO, U2 RP2040-Connect

Commit message: Added GY87 and DC DC Buck
Parts:
- added U10: ~, MicroMouse_2025_v2:GY-87, symbol MicroMouse_2025_v2:GY-87
- added U9: ~, MicroMouse_2025_v2:DC-DC 5V3A BEC, symbol MicroMouse_2025_v2:DC-DC_5V_3A_BEC
Other:
- moved on the sheet: D1, D2, D3, D4, J1, R1, S1, S2, S3
